File: GarageDoorOpener.sch (KiCad schematic (older format))
At the start: 10 parts

Commit message: small amount of work done, added some documentation
Parts:
- added C?: 1uF 10V, symbol Device:C
- added D? (x2): LED, symbol Device:LED
- added R? (x2): 10K, symbol Device:R
- added R? (x2): 1K, symbol Device:R
- C? (x3): value 47uF -> 47uF 10V
- C?: value 1uF -> 1uF 10V
Connections:
- net REED_SW1_IN is gone; now on net REED_SW1: J?.1 (Pin_1)
- net REED_SW2_IN is gone; now on net REED_SW2: J?.1 (Pin_1)
- net CONNECTIVITY_LED: now also R?.1
- net GND: now also C?.2
- net REED_SW1: now also R?.2
- net REED_SW2: now also R?.2
- net STATUS_LED: now also R?.1
- net +3V3: now reaches U?.2 (3.3V)
- net +3V3: now also C?.1, R?.1, R?.1
- new net: D?.2 (A), R?.2 (x2)
Other:
- note added: "NOTE: MAINTAIN 0.6mm MINIMUM DISTANCE BETWEEN AC TRACES"
- note removed: "NOTE: MAINTAIN XXmm DISTANCE BETWEEN AC TRACES"
- moved on the sheet: C?, J?
Changed lines of the file:
@@
 Wire Wire Line
 	2000 1775 1575 1775
-Text Notes 1000 2050 0    50   ~ 0
-NOTE: MAINTAIN XXmm DISTANCE BETWEEN AC TRACES
+Text Notes 775  2025 0    50   ~ 0
+NOTE: MAINTAIN 0.6mm MINIMUM DISTANCE BETWEEN AC TRACES
 $Comp
 L power:GND #PWR?
@@
 	3000 1625 3550 1625
 Wire Wire Line
-	4425 1625 4425 1475
+	4650 1625 4650 1475
 $Comp
 L power:+5V #PWR?
 U 1 1 5EA80065
-P 4425 1475
-F 0 "#PWR?" H 4425 1325 50  0001 C CNN
-F 1 "+5V" H 4440 1648 50  0000 C CNN
-F 2 "" H 4425 1475 50  0001 C CNN
-F 3 "" H 4425 1475 50  0001 C CNN
-	1    4425 1475
+P 4650 1475
+F 0 "#PWR?" H 4650 1325 50  0001 C CNN
+F 1 "+5V" H 4665 1648 50  0000 C CNN
+F 2 "" H 4650 1475 50  0001 C CNN
+F 3 "" H 4650 1475 50  0001 C CNN
+	1    4650 1475
 	1    0    0    -1
 $EndComp
@@
 P 3550 1875
 F 0 "C?" H 3575 1950 50  0000 L CNN
-F 1 "47uF" H 3575 1775 50  0000 L CNN
+F 1 "47uF 10V" H 3350 1775 50  0000 L CNN
 F 2 "" H 3588 1725 50  0001 C CNN
 F 3 "~" H 3550 1875 50  0001 C CNN
@@
 L device:C C?
 U 1 1 5EA8195E
-P 3900 1875
-F 0 "C?" H 3925 1950 50  0000 L CNN
-F 1 "47uF" H 3925 1775 50  0000 L CNN
-F 2 "" H 3938 1725 50  0001 C CNN
-F 3 "~" H 3900 1875 50  0001 C CNN
-	1    3900 1875
+P 4000 1875
+F 0 "C?" H 4025 1950 50  0000 L CNN
+F 1 "47uF 10V" H 3800 1775 50  0000 L CNN
+F 2 "" H 4038 1725 50  0001 C CNN
+F 3 "~" H 4000 1875 50  0001 C CNN
+	1    4000 1875
 	1    0    0    -1
 $EndComp
@@
 L device:C C?
 U 1 1 5EA81F80
-P 4250 1875
-F 0 "C?" H 4275 1950 50  0000 L CNN
-F 1 "47uF" H 4275 1775 50  0000 L CNN
-F 2 "" H 4288 1725 50  0001 C CNN
-F 3 "~" H 4250 1875 50  0001 C CNN
-	1    4250 1875
+P 4475 1875
+F 0 "C?" H 4500 1950 50  0000 L CNN
+F 1 "47uF 10V" H 4275 1775 50  0000 L CNN
+F 2 "" H 4513 1725 50  0001 C CNN
+F 3 "~" H 4475 1875 50  0001 C CNN
+	1    4475 1875
 	1    0    0    -1
 $EndComp
@@
 	3250 2100 3250 2175
 Wire Wire Line
-	3550 2100 3900 2100
-Wire Wire Line
-	4250 2100 4250 2025
+	3550 2100 4000 2100
+Wire Wire Line
+	4475 2100 4475 2025
 Connection ~ 3550 2100
 Wire Wire Line
-	3900 2025 3900 2100
-Connection ~ 3900 2100
-Wire Wire Line
-	3900 2100 4250 2100
-Wire Wire Line
-	4250 1725 4250 1625
-Connection ~ 4250 1625
-Wire Wire Line
-	4250 1625 4425 1625
-Wire Wire Line
-	3900 1725 3900 1625
-Connection ~ 3900 1625
-Wire Wire Line
-	3900 1625 4250 1625
+	4000 2025 4000 2100
+Connection ~ 4000 2100
+Wire Wire Line
+	4000 2100 4475 2100
+Wire Wire Line
+	4475 1725 4475 1625
+Connection ~ 4475 1625
+Wire Wire Line
+	4475 1625 4650 1625
+Wire Wire Line
+	4000 1725 4000 1625
+Connection ~ 4000 1625
+Wire Wire Line
+	4000 1625 4475 1625
 Wire Wire Line
 	3550 1725 3550 1625
 Connection ~ 3550 1625
 Wire Wire Line
-	3550 1625 3900 1625
+	3550 1625 4000 1625
 Wire Notes Line
 	4875 950  4875 2525
@@
 $EndComp
 Wire Wire Line
-	5825 3175 5825 1875
+	5825 3175 5825 2175
 Wire Wire Line
 	5825 1875 5925 1875
@@
 P 9975 1750
 F 0 "C?" H 10090 1796 50  0000 L CNN
-F 1 "1uF" H 10090 1705 50  0000 L CNN
+F 1 "1uF 10V" H 9825 1650 50  0000 L CNN
 F 2 "" H 10013 1600 50  0001 C CNN
 F 3 "~" H 9975 1750 50  0001 C CNN
@@
 L conn:Conn_01x02 J?
 U 1 1 5EA990EC
-P 9825 3975
-F 0 "J?" H 9905 3967 50  0000 L CNN
-F 1 "Conn_01x02" H 9905 3876 50  0000 L CNN
-F 2 "" H 9825 3975 50  0001 C CNN
-F 3 "~" H 9825 3975 50  0001 C CNN
-	1    9825 3975
+P 9825 5900
+F 0 "J?" H 9905 5892 50  0000 L CNN
+F 1 "Conn_01x02" H 9905 5801 50  0000 L CNN
+F 2 "" H 9825 5900 50  0001 C CNN
+F 3 "~" H 9825 5900 50  0001 C CNN
+	1    9825 5900
 	1    0    0    -1
 $EndComp
@@
 	1    0    0    -1
 $EndComp
-Text Notes 9725 3800 0    50   ~ 0
+Text Notes 9725 5725 0    50   ~ 0
 RELAY
 Text Notes 9650 4375 0    50   ~ 0
@@
 Text Notes 9625 4950 0    50   ~ 0
 REED SW2
-Text HLabel 9400 4550 0    50   Input ~ 0
-REED_SW1_IN
-Text HLabel 9400 5100 0    50   Input ~ 0
-REED_SW2_IN
-Wire Wire Line
-	9400 4550 9625 4550
+Text HLabel 8950 4550 0    50   Input ~ 0
+REED_SW1
+Text HLabel 8950 5100 0    50   Input ~ 0
+REED_SW2
+Wire Wire Line
+	8950 4550 9150 4550
 Wire Wire Line
 	9625 5100 9400 5100
@@
 	9525 4650 9525 5200
 Connection ~ 9525 5200
+$Comp
+L Device:R R?
+U 1 1 5EA94A9E
+P 9150 4300
+F 0 "R?" H 9220 4346 50  0000 L CNN
+F 1 "10K" V 9150 4225 50  0000 L CNN
+F 2 "" V 9080 4300 50  0001 C CNN
+F 3 "~" H 9150 4300 50  0001 C CNN
+	1    9150 4300
+	1    0    0    -1
+$EndComp
+$Comp
+L Device:R R?
+U 1 1 5EA954E2
+P 9400 4300
+F 0 "R?" H 9470 4346 50  0000 L CNN
+F 1 "10K" V 9400 4225 50  0000 L CNN
+F 2 "" V 9330 4300 50  0001 C CNN
+F 3 "~" H 9400 4300 50  0001 C CNN
+	1    9400 4300
+	1    0    0    -1
+$EndComp
+Connection ~ 9400 5100
+Wire Wire Line
+	9400 5100 8950 5100
+Wire Wire Line
+	9400 4450 9400 5100
+Wire Wire Line
+	9150 4450 9150 4550
+Connection ~ 9150 4550
+Wire Wire Line
+	9150 4550 9625 4550
+Wire Wire Line
+	9150 4000 9150 4050
+Wire Wire Line
+	9150 4050 9400 4050
+Wire Wire Line
+	9400 4050 9400 4150
+Connection ~ 9150 4050
+Wire Wire Line
+	9150 4050 9150 4150
+$Comp
+L FeatherWing_KC5-cache:+3.3V #PWR?
+U 1 1 5EA9BBC7
+P 5575 1375
+F 0 "#PWR?" H 5575 1225 50  0001 C CNN
+F 1 "+3.3V" H 5590 1548 50  0000 C CNN
+F 2 "" H 5575 1375 50  0001 C CNN
+F 3 "" H 5575 1375 50  0001 C CNN
+	1    5575 1375
+	1    0    0    -1
+$EndComp
+Wire Wire Line
+	5575 1375 5575 1675
+Wire Wire Line
+	5575 1675 5925 1675
+$Comp
+L Device:C C?
+U 1 1 5EA9DB02
+P 5575 1925
+F 0 "C?" H 5690 1971 50  0000 L CNN
+F 1 "1uF 10V" H 5425 1825 50  0000 L CNN
+F 2 "" H 5613 1775 50  0001 C CNN
+F 3 "~" H 5575 1925 50  0001 C CNN
+	1    5575 1925
+	1    0    0    -1
+$EndComp
+Wire Wire Line
+	5575 1775 5575 1675
+Connection ~ 5575 1675
+Wire Wire Line
+	5575 2075 5575 2175
+Wire Wire Line
+	5575 2175 5825 2175
+Connection ~ 5825 2175
+Wire Wire Line
+	5825 2175 5825 1875
+$Comp
+L FeatherWing_KC5-cache:+3.3V #PWR?
+U 1 1 5EAA0B2A
+P 9150 4000
+F 0 "#PWR?" H 9150 3850 50  0001 C CNN
+F 1 "+3.3V" H 9165 4173 50  0000 C CNN
+F 2 "" H 9150 4000 50  0001 C CNN
+F 3 "" H 9150 4000 50  0001 C CNN
+	1    9150 4000
+	1    0    0    -1
+$EndComp
+$Comp
+L Device:LED D?
+U 1 1 5EAA1E6A
+P 4675 5650
+F 0 "D?" V 4714 5532 50  0000 R CNN
+F 1 "LED" V 4623 5532 50  0000 R CNN
+F 2 "" H 4675 5650 50  0001 C CNN
+F 3 "~" H 4675 5650 50  0001 C CNN
+	1    4675 5650
+	0    -1   -1   0
+$EndComp
+$Comp
+L Device:LED D?
+U 1 1 5EAA25FE
+P 5250 5650
+F 0 "D?" V 5289 5532 50  0000 R CNN
+F 1 "LED" V 5198 5532 50  0000 R CNN
+F 2 "" H 5250 5650 50  0001 C CNN
+F 3 "~" H 5250 5650 50  0001 C CNN
+	1    5250 5650
+	0    -1   -1   0
+$EndComp
+$Comp
+L Device:R R?
+U 1 1 5EAA2AA0
+P 4675 5175
+F 0 "R?" H 4745 5221 50  0000 L CNN
+F 1 "1K" V 4675 5125 50  0000 L CNN
+F 2 "" V 4605 5175 50  0001 C CNN
+F 3 "~" H 4675 5175 50  0001 C CNN
+	1    4675 5175
+	1    0    0    -1
+$EndComp
+$Comp
+L Device:R R?
+U 1 1 5EAA320D
+P 5250 5175
+F 0 "R?" H 5320 5221 50  0000 L CNN
+F 1 "1K" V 5250 5125 50  0000 L CNN
+F 2 "" V 5180 5175 50  0001 C CNN
+F 3 "~" H 5250 5175 50  0001 C CNN
+	1    5250 5175
+	1    0    0    -1
+$EndComp
+Wire Wire Line
+	5250 5325 5250 5500
+Wire Wire Line
+	4675 5325 4675 5500
+Text HLabel 4675 4875 1    50   Input ~ 0
+CONNECTIVITY_LED
+Wire Wire Line
+	4675 4875 4675 5025
+Text HLabel 5250 4825 1    50   Input ~ 0
+STATUS_LED
+Wire Wire Line
+	5250 4825 5250 5025
 $EndSCHEMATC

Commit message: first pass on the schematic done
Parts:
- added Q?: DMG1012T-7, symbol Device:Q_NMOS_GSD
- added R?: 649, symbol Device:R
- added R?: 10K, symbol Device:R
- added U?: CPC1002N, symbol Global_Parts:CPC1002N
Connections:
- net +3V3: now also R?.2
- net GND: now also D?.1 (K), D?.1 (K), Q?.2 (S), R?.1
- net RELAY_CTRL: now also Q?.1 (G), R?.2
- net at J?.1 (Pin_1): now also U?.4
- net at J?.2 (Pin_2): now also U?.3
- new net: Q?.3 (D), U?.2
- new net: R?.1, U?.1
- no-connect marks 1 -> 20
Other:
- note added: "(3.3V-1.2V)/3mA = 700 ohms\n(3.3V-1.5V)/3mA = 600 ohms (worst case Vf)"
- note added: "2mA minimum LED current\n1.2V LED Vf"
- note added: "Reed Switch Input"
- note added: "Relay Switch Control"
- note added: "Status LEDs"
- moved on the sheet: D?, J?, R?
