File: Hardware/GarageDoorOpener.sch (KiCad schematic (older format))
At the start: 21 parts

Commit message: schematic slightly updated (footprint association) PCB started
Parts:
- added H1, H2, H3, H4: MountingHole, MountingHole:MountingHole_3.2mm_M3, symbol mechanical:MountingHole
- C1, C2, C3: renamed from C?; footprint (none) -> Capacitor_SMD:C_1206_3216Metric
- C4, C5: renamed from C?; footprint (none) -> Capacitor_SMD:C_0603_1608Metric
- D1, D2: renamed from D?; footprint (none) -> LED_SMD:LED_0805_2012Metric
- J1: renamed from J?; footprint (none) -> Connector_Phoenix_MC:PhoenixContact_MCV_1,5_2-G-3.5_1x02_P3.50mm_Vertical
- J2, J3, J4: renamed from J?; footprint (none) -> Connector_JST:JST_PH_S2B-PH-K_1x02_P2.00mm_Horizontal
- Q1: renamed from Q?; footprint (none) -> Package_TO_SOT_SMD:SOT-523
- R1, R2, R3, R4, R5, R6: renamed from R?; footprint (none) -> Resistor_SMD:R_0603_1608Metric
- U1, U2: renamed from U?; footprint (none) -> Package_SO:SOP-4_3.8x4.1mm_P2.54mm
- gave numbers to parts that had none: 1
Other:
- note added: "M3 Mounting Holes"

Commit message: scope creep is great, decided to expand on the project a bit, Rev1b
Parts:
- removed C1, C2, C3: 47uF 10V, Capacitor_SMD:C_1206_3216Metric, symbol device:C
- removed J1: Conn_01x02, Connector_Phoenix_MC:PhoenixContact_MCV_1,5_2-G-3.5_1x02_P3.50mm_Vertical, symbol conn:Conn_01x02
- removed J2, J3, J4: Conn_01x02, Connector_JST:JST_PH_S2B-PH-K_1x02_P2.00mm_Horizontal, symbol conn:Conn_01x02
- removed R4: 649, Resistor_SMD:R_0603_1608Metric, symbol Device:R
- removed U1: RAC15-05SK, Package_SO:SOP-4_3.8x4.1mm_P2.54mm, symbol Global_Parts:RAC15-05SK
- removed U2: CPC1002N, Package_SO:SOP-4_3.8x4.1mm_P2.54mm, symbol Global_Parts:CPC1002N
- added C1, C2, C3: 4.7uF 50V, symbol Device:C
- added C10, C9: 22uF 10V, symbol Device:C
- added C11: 4.7uF 10V, symbol Device:C
- added C12: 0.1uF 10V, symbol Device:C
- added C13: 10uF 10V, symbol Device:C
- added C4: 0.1uF 50V, symbol Device:C
- added C7: 0.1uF, symbol Device:C
- added C8: 100pF 10V, symbol Device:C
- added J1: Conn_01x04, symbol conn:Conn_01x04
- added J2: RJ45, symbol Connector:RJ45
- added L1: 3.3uH, symbol Device:L
- added R10: 73.2K, symbol Device:R
- added R11: 10K, symbol Device:R
- added R12, R13: 4.7K, Resistor_SMD:R_0603_1608Metric, symbol Device:R
- added R14, R15, R2, R7, R9: 10K, Resistor_SMD:R_0603_1608Metric, symbol Device:R
- added R8: 20K, symbol Device:R
- added U2: TPS56637, MODULE, symbol Global_Parts:TPS56637
- added U4: VL53L1X, MODULE, symbol Global_Parts:VL53L1X
- added UU3: CPC1002N, Package_SO:SOP-4_3.8x4.1mm_P2.54mm, symbol Global_Parts:CPC1002N
- R3: value 10K -> 649
- R5: footprint Resistor_SMD:R_0603_1608Metric -> (none)
- R6: value 10K -> 100K; footprint Resistor_SMD:R_0603_1608Metric -> (none)
- renumbered C4 to C6, R2 to R4, U3 to U1
Connections:
- net +3V3: now also R3.2, C11.1, C12.1, R12.1, R13.1, R14.1, R15.1, R7.1, R9.1, U4.1 (AVDD_VCSEL), U4.11 (AVDD); no longer R5.1, R6.1
- net +5V: now also R6.1, C10.2, C13.1, C9.2, J1.1 (Pin_1), L1.2, R10.2, R8.2
- net CONNECTIVITY_LED: now also U1.9 (A4/PWM); no longer U1.22 (D5/PWM)
- net GND: now also C1.2, C10.1, C11.2, C12.2, C13.2, C2.2, C3.2, C4.2, C9.1, J1.4 (Pin_4), J2.2, J2.6, J2.8, R11.1, R2.1, U2.10 (MODE), U2.3 (AGND), U2.9 (PGND), U4.12 (GND), U4.2 (AVSS_VCSEL), U4.3 (GND), U4.4 (GND), U4.6 (GND), U4.8 (DNC); no longer R3.1
- net REED_SW1: now also J2.7, R7.2; no longer R5.2
- net REED_SW2: now also J2.5, R9.2; no longer R6.2
- net STATUS_LED: now also U1.8 (A3/PWM); no longer U1.21 (D4/PWM/SPI1_MISO)
- net LED_STRIP_CLK: now reaches U1.11 (SPI_SCLK)
- net LED_STRIP_CLK: now also J1.2 (Pin_2)
- net LED_STRIP_DATA: now reaches U1.12 (SPI_MOSI)
- net LED_STRIP_DATA: now also J1.3 (Pin_3)
- net SENSOR_I2C_SDA: now reaches U1.17 (I2C_SDA)
- net SENSOR_I2C_SDA: now also R12.2, U4.9 (SDA)
- net SENSOR_I2C_SCL: now reaches U1.18 (I2C_SCL)
- net SENSOR_I2C_SCL: now also R13.2, U4.10 (SCL)
- net SENSOR_INT: now reaches U1.19 (D2/PWM/SPI1_SCLK/UART_RTS)
- net SENSOR_INT: now also R14.2, U4.7 (GPIO1_INT)
- net SENSOR_SHUTDOWN: now reaches U1.20 (D3/PWM/SPI1_MOSI/UART_CTS)
- net SENSOR_SHUTDOWN: now also R15.2, U4.5 (XSHUT)
- net at Q1.3 (D): now also UU3.2
- net RELAY_CTRL renamed RELAY_CTRL1
- net RELAY_CTRL1: now also R2.2; no longer R3.2
- new net: R3.1, UU3.1
- new net: R5.2, U2.1 (EN)
- new net: C8.1, R10.1, R11.2, U2.2 (FB)
- new net: R6.2, U2.4 (PG)
- new net: C7.1, L1.1, U2.6 (SW)
- new net: C7.2, U2.7 (BOOT)
- new net: C8.2, R8.1
- new net +24V: C1.1, C2.1, C3.1, C4.1, J2.1, R5.1, U2.8 (VIN)
- new net Relay_Ouput1: J2.3, UU3.4
- new net Relay_Ouput2: J2.4, UU3.3
- no-connect marks 20 -> 15
Other:
- note added: "24V to 5V@4A Buck Regulator"
- note added: "Board Input/output"
- note added: "Distance Sensor"
- note added: "LED Strip Header\n"
- note added: "Reed Switch Input Block 1"
- note added: "Relay Control Block 1"
- note removed: "120V to 5V AC-DC Converter"
- note removed: "NOTE: MAINTAIN 0.6mm MINIMUM DISTANCE BETWEEN AC TRACES"
- note removed: "Reed Switch Input"
- note removed: "Relay Switch Control"
- moved on the sheet: C5, C6, D1, D2, H1, H2, H3, H4, R1, R4, U1
