File: Hardware/ControlBoard/GarageDoorOpener.sch (KiCad schematic (older format))
At the start: 42 parts, among them J1 Conn_01x04, J2 RJ45, Q1 DMG1012T-7, U1 Argon/Boron, U2 TPS56637, U4 VL53L1X

Commit message: I moved files again, added the power board schematic, working on BoM
Parts:
- added R16, R17, R18, R19, R20, R21: 0, symbol Device:R
- renumbered UU3 to U3
Connections:
- wire segments 187 -> 193
Changed lines of the file:
@@
 $EndComp
 $Comp
-L Global_Parts:CPC1002N UU3
+L Global_Parts:CPC1002N U3
 U 1 1 5EB006DB
 P 2300 4050
-AR Path="/5EB006DB" Ref="UU3"  Part="1"
+AR Path="/5EB006DB" Ref="U3"  Part="1"
 AR Path="/5EB107FD/5EB006DB" Ref="U?"  Part="1"
-F 0 "UU3" H 2300 4175 50  0000 C CNN
+F 0 "U3" H 2300 4175 50  0000 C CNN
 F 1 "CPC1002N" H 2300 4084 50  0000 C CNN
 F 2 "Package_SO:SOP-4_3.8x4.1mm_P2.54mm" H 2300 4050 50  0001 C CNN
@@
 	-1   0    0    1
 $EndComp
-Text HLabel 9575 2825 0    50   Input ~ 0
+Text HLabel 9175 2825 0    50   Input ~ 0
 REED_SW2_IN
-Text HLabel 9575 2925 0    50   Input ~ 0
+Text HLabel 9175 2925 0    50   Input ~ 0
 REED_SW2_GND
-Text HLabel 9575 3025 0    50   Input ~ 0
+Text HLabel 9175 3025 0    50   Input ~ 0
 REED_SW1_IN
-Text HLabel 9575 3125 0    50   Input ~ 0
+Text HLabel 9175 3125 0    50   Input ~ 0
 REED_SW1_GND
-Text HLabel 9575 2625 0    50   Input ~ 0
+Text HLabel 9175 2625 0    50   Input ~ 0
 Relay_Ouput1
-Text HLabel 9575 2725 0    50   Input ~ 0
+Text HLabel 9175 2725 0    50   Input ~ 0
 Relay_Ouput2
 $Comp
@@
 	8250 2100 10975 2100
 Wire Wire Line
-	9575 3125 9850 3125
-Wire Wire Line
-	9850 3025 9575 3025
-Wire Wire Line
-	9575 2925 9850 2925
-Wire Wire Line
-	9850 2825 9575 2825
-Wire Wire Line
-	9575 2725 9850 2725
-Wire Wire Line
-	9850 2625 9575 2625
+	9650 3125 9850 3125
+Wire Wire Line
+	9850 3025 9650 3025
+Wire Wire Line
+	9650 2925 9850 2925
+Wire Wire Line
+	9850 2825 9650 2825
+Wire Wire Line
+	9650 2725 9850 2725
+Wire Wire Line
+	9850 2625 9650 2625
 $Comp
 L Device:R R?
@@
 Text Notes 3050 7175 0    50   ~ 0
 24V to 5V@4A Buck Regulator
+Wire Wire Line
+	9350 2625 9175 2625
+Wire Wire Line
+	9350 2725 9175 2725
+Wire Wire Line
+	9350 2825 9175 2825
+Wire Wire Line
+	9350 2925 9175 2925
+Wire Wire Line
+	9350 3025 9175 3025
+$Comp
+L Device:R R21
+U 1 1 5EB42735
+P 9500 3125
+F 0 "R21" V 9550 2975 50  0000 C CNN
+F 1 "0" V 9500 3125 50  0000 C CNN
+F 2 "" V 9430 3125 50  0001 C CNN
+F 3 "~" H 9500 3125 50  0001 C CNN
+	1    9500 3125
+	0    1    1    0
+$EndComp
+Wire Wire Line
+	9350 3125 9175 3125
+$Comp
+L Device:R R20
+U 1 1 5EB4D6BA
+P 9500 3025
+F 0 "R20" V 9550 2875 50  0000 C CNN
+F 1 "0" V 9500 3025 50  0000 C CNN
+F 2 "" V 9430 3025 50  0001 C CNN
+F 3 "~" H 9500 3025 50  0001 C CNN
+	1    9500 3025
+	0    1    1    0
+$EndComp
+$Comp
+L Device:R R19
+U 1 1 5EB4D95E
+P 9500 2925
+F 0 "R19" V 9550 2775 50  0000 C CNN
+F 1 "0" V 9500 2925 50  0000 C CNN
+F 2 "" V 9430 2925 50  0001 C CNN
+F 3 "~" H 9500 2925 50  0001 C CNN
+	1    9500 2925
+	0    1    1    0
+$EndComp
+$Comp
+L Device:R R18
+U 1 1 5EB4DC76
+P 9500 2825
+F 0 "R18" V 9550 2675 50  0000 C CNN
+F 1 "0" V 9500 2825 50  0000 C CNN
+F 2 "" V 9430 2825 50  0001 C CNN
+F 3 "~" H 9500 2825 50  0001 C CNN
+	1    9500 2825
+	0    1    1    0
+$EndComp
+$Comp
+L Device:R R17
+U 1 1 5EB4DED5
+P 9500 2725
+F 0 "R17" V 9550 2575 50  0000 C CNN
+F 1 "0" V 9500 2725 50  0000 C CNN
+F 2 "" V 9430 2725 50  0001 C CNN
+F 3 "~" H 9500 2725 50  0001 C CNN
+	1    9500 2725
+	0    1    1    0
+$EndComp
+$Comp
+L Device:R R16
+U 1 1 5EB4E167
+P 9500 2625
+F 0 "R16" V 9550 2475 50  0000 C CNN
+F 1 "0" V 9500 2625 50  0000 C CNN
+F 2 "" V 9430 2625 50  0001 C CNN
+F 3 "~" H 9500 2625 50  0001 C CNN
+	1    9500 2625
+	0    1    1    0
+$EndComp
 $EndSCHEMATC

Commit message: Schematics done, PCBs have components dropped in and BoM finished
Parts:
- C1, C10, C2, C3, C9: footprint (none) -> Capacitor_SMD:C_0805_2012Metric
- C11: footprint (none) -> Capacitor_SMD:C_0603_1608Metric
- C12: value 0.1uF 10V -> 0.1uF 16V; footprint (none) -> Capacitor_SMD:C_0603_1608Metric
- C13: value 10uF 10V -> 4.7uF 10V; footprint (none) -> Capacitor_SMD:C_0603_1608Metric
- C4, C8: footprint (none) -> Capacitor_SMD:C_0201_0603Metric
- C7: value 0.1uF -> 0.1uF 16V; footprint (none) -> Capacitor_SMD:C_0603_1608Metric
- D1: value LED -> GREEN_LED
- D2: value LED -> RED_LED
- J1: footprint (none) -> Connector_JST:JST_PH_B4B-PH-K_1x04_P2.00mm_Vertical
- J2: footprint (none) -> Connector_RJ:RJ45_Amphenol_54602-x08_Horizontal
- L1: footprint (none) -> Inductor_SMD:L_Taiyo-Yuden_NR-40xx
- R1: value 1K -> 649
- R10, R11, R16, R17, R18, R19, R20, R21, R5, R8: footprint (none) -> Resistor_SMD:R_0603_1608Metric
- R6: value 100K -> 10K; footprint (none) -> Resistor_SMD:R_0603_1608Metric
- U1: footprint MODULE -> Global_Parts:ParticleBoron
- U2: footprint MODULE -> Global_Parts:TPS56637RPAR
- U4: footprint MODULE -> Global_Parts:VL53L1CXV0FY_1
Changed lines of the file:
@@
 F 0 "U1" H 5412 2965 50  0000 C CNN
 F 1 "Argon/Boron" H 5412 2874 50  0000 C CNN
-F 2 "MODULE" H 5400 1050 50  0001 C CNN
+F 2 "Global_Parts:ParticleBoron" H 5400 1050 50  0001 C CNN
 F 3 "DOCUMENTATION" H 5225 950 50  0001 C CNN
 	1    5400 1975
@@
 P 1275 2425
 F 0 "D1" V 1314 2307 50  0000 R CNN
-F 1 "LED" V 1223 2307 50  0000 R CNN
+F 1 "GREEN_LED" H 1475 2525 50  0000 R CNN
 F 2 "LED_SMD:LED_0805_2012Metric" H 1275 2425 50  0001 C CNN
 F 3 "~" H 1275 2425 50  0001 C CNN
@@
 P 1850 2425
 F 0 "D2" V 1889 2307 50  0000 R CNN
-F 1 "LED" V 1798 2307 50  0000 R CNN
+F 1 "RED_LED" H 1950 2525 50  0000 R CNN
 F 2 "LED_SMD:LED_0805_2012Metric" H 1850 2425 50  0001 C CNN
 F 3 "~" H 1850 2425 50  0001 C CNN
@@
 P 1275 2000
 F 0 "R1" H 1345 2046 50  0000 L CNN
-F 1 "1K" V 1275 1950 50  0000 L CNN
+F 1 "649" V 1275 1925 50  0000 L CNN
 F 2 "Resistor_SMD:R_0603_1608Metric" V 1205 2000 50  0001 C CNN
 F 3 "~" H 1275 2000 50  0001 C CNN
@@
 F 0 "J1" H 10305 1392 50  0000 L CNN
 F 1 "Conn_01x04" H 10305 1301 50  0000 L CNN
-F 2 "" H 10225 1400 50  0001 C CNN
+F 2 "Connector_JST:JST_PH_B4B-PH-K_1x04_P2.00mm_Vertical" H 10225 1400 50  0001 C CNN
 F 3 "~" H 10225 1400 50  0001 C CNN
 	1    10225 1400
@@
 P 8825 1450
 F 0 "C13" H 8850 1550 50  0000 L CNN
-F 1 "10uF 10V" H 8625 1350 50  0000 L CNN
-F 2 "" H 8863 1300 50  0001 C CNN
+F 1 "4.7uF 10V" H 8625 1350 50  0000 L CNN
+F 2 "Capacitor_SMD:C_0603_1608Metric" H 8863 1300 50  0001 C CNN
 F 3 "~" H 8825 1450 50  0001 C CNN
 	1    8825 1450
@@
 F 0 "U4" H 9750 5640 50  0000 C CNN
 F 1 "VL53L1X" H 9750 5549 50  0000 C CNN
-F 2 "MODULE" H 10100 4675 50  0001 C CNN
+F 2 "Global_Parts:VL53L1CXV0FY_1" H 10100 4675 50  0001 C CNN
 F 3 "DOCUMENTATION" H 9950 4750 50  0001 C CNN
 	1    9750 5025
@@
 F 0 "C11" H 7550 4325 50  0000 L CNN
 F 1 "4.7uF 10V" H 7300 4125 50  0000 L CNN
-F 2 "" H 7563 4075 50  0001 C CNN
+F 2 "Capacitor_SMD:C_0603_1608Metric" H 7563 4075 50  0001 C CNN
 F 3 "~" H 7525 4225 50  0001 C CNN
 	1    7525 4225
@@
 P 7975 4225
 F 0 "C12" H 8000 4325 50  0000 L CNN
-F 1 "0.1uF 10V" H 7750 4125 50  0000 L CNN
-F 2 "" H 8013 4075 50  0001 C CNN
+F 1 "0.1uF 16V" H 7750 4125 50  0000 L CNN
+F 2 "Capacitor_SMD:C_0603_1608Metric" H 8013 4075 50  0001 C CNN
 F 3 "~" H 7975 4225 50  0001 C CNN
 	1    7975 4225
@@
 F 0 "U2" H 3175 7290 50  0000 C CNN
 F 1 "TPS56637" H 3175 7199 50  0000 C CNN
-F 2 "MODULE" H 3475 6375 50  0001 C CNN
+F 2 "Global_Parts:TPS56637RPAR" H 3475 6375 50  0001 C CNN
 F 3 "DOCUMENTATION" H 3325 6475 50  0001 C CNN
 	1    3175 6725
@@
 P 4075 6425
 F 0 "C7" V 3823 6425 50  0000 C CNN
-F 1 "0.1uF" V 3914 6425 50  0000 C CNN
-F 2 "" H 4113 6275 50  0001 C CNN
+F 1 "0.1uF 16V" V 3914 6425 50  0000 C CNN
+F 2 "Capacitor_SMD:C_0603_1608Metric" H 4113 6275 50  0001 C CNN
 F 3 "~" H 4075 6425 50  0001 C CNN
 	1    4075 6425
@@
 F 0 "L1" V 4840 6425 50  0000 C CNN
 F 1 "3.3uH" V 4749 6425 50  0000 C CNN
-F 2 "" H 4650 6425 50  0001 C CNN
+F 2 "Inductor_SMD:L_Taiyo-Yuden_NR-40xx" H 4650 6425 50  0001 C CNN
 F 3 "~" H 4650 6425 50  0001 C CNN
 	1    4650 6425
@@
 P 4650 6625
 F 0 "R6" V 4550 6625 50  0000 C CNN
-F 1 "100K" V 4650 6625 50  0000 C CNN
-F 2 "" V 4580 6625 50  0001 C CNN
+F 1 "10K" V 4650 6625 50  0000 C CNN
+F 2 "Resistor_SMD:R_0603_1608Metric" V 4580 6625 50  0001 C CNN
 F 3 "~" H 4650 6625 50  0001 C CNN
 	1    4650 6625
@@
 F 0 "R10" V 5650 6750 50  0000 C CNN
 F 1 "73.2K" V 5750 6750 50  0000 C CNN
-F 2 "" V 5680 6750 50  0001 C CNN
+F 2 "Resistor_SMD:R_0603_1608Metric" V 5680 6750 50  0001 C CNN
 F 3 "~" H 5750 6750 50  0001 C CNN
 	1    5750 6750
@@
 F 0 "R11" V 5650 7150 50  0000 C CNN
 F 1 "10K" V 5750 7150 50  0000 C CNN
-F 2 "" V 5680 7150 50  0001 C CNN
+F 2 "Resistor_SMD:R_0603_1608Metric" V 5680 7150 50  0001 C CNN
 F 3 "~" H 5750 7150 50  0001 C CNN
 	1    5750 7150
@@
 F 0 "R8" V 5250 6550 50  0000 C CNN
 F 1 "20K" V 5350 6550 50  0000 C CNN
-F 2 "" V 5280 6550 50  0001 C CNN
+F 2 "Resistor_SMD:R_0603_1608Metric" V 5280 6550 50  0001 C CNN
 F 3 "~" H 5350 6550 50  0001 C CNN
 	1    5350 6550
@@
 F 0 "C8" H 5100 6700 50  0000 R CNN
 F 1 "100pF 10V" H 5375 6875 50  0000 R CNN
-F 2 "" H 5163 6625 50  0001 C CNN
+F 2 "Capacitor_SMD:C_0201_0603Metric" H 5163 6625 50  0001 C CNN
 F 3 "~" H 5125 6775 50  0001 C CNN
 	1    5125 6775
@@
 F 0 "C10" H 6410 6829 50  0000 R CNN
 F 1 "22uF 10V" H 6725 6975 50  0000 R CNN
-F 2 "" H 6563 6725 50  0001 C CNN
+F 2 "Capacitor_SMD:C_0805_2012Metric" H 6563 6725 50  0001 C CNN
 F 3 "~" H 6525 6875 50  0001 C CNN
 	1    6525 6875
@@
 F 0 "C4" H 2000 6750 50  0000 L CNN
 F 1 "0.1uF 50V" V 1825 6450 50  0000 L CNN
-F 2 "" H 2013 6500 50  0001 C CNN
+F 2 "Capacitor_SMD:C_0201_0603Metric" H 2013 6500 50  0001 C CNN
 F 3 "~" H 1975 6650 50  0001 C CNN
 	1    1975 6650
@@
 F 0 "C3" H 1650 6750 50  0000 L CNN
 F 1 "4.7uF 50V" V 1500 6450 50  0000 L CNN
-F 2 "" H 1663 6500 50  0001 C CNN
+F 2 "Capacitor_SMD:C_0805_2012Metric" H 1663 6500 50  0001 C CNN
 F 3 "~" H 1625 6650 50  0001 C CNN
 	1    1625 6650
@@
 F 0 "C2" H 1325 6750 50  0000 L CNN
 F 1 "4.7uF 50V" V 1175 6450 50  0000 L CNN
-F 2 "" H 1338 6500 50  0001 C CNN
+F 2 "Capacitor_SMD:C_0805_2012Metric" H 1338 6500 50  0001 C CNN
 F 3 "~" H 1300 6650 50  0001 C CNN
 	1    1300 6650
@@
 F 0 "C1" H 1000 6750 50  0000 L CNN
 F 1 "4.7uF 50V" V 850 6450 50  0000 L CNN
-F 2 "" H 1013 6500 50  0001 C CNN
+F 2 "Capacitor_SMD:C_0805_2012Metric" H 1013 6500 50  0001 C CNN
 F 3 "~" H 975 6650 50  0001 C CNN
 	1    975  6650
@@
 F 0 "C9" H 5985 6829 50  0000 R CNN
 F 1 "22uF 10V" H 6300 6975 50  0000 R CNN
-F 2 "" H 6138 6725 50  0001 C CNN
+F 2 "Capacitor_SMD:C_0805_2012Metric" H 6138 6725 50  0001 C CNN
 F 3 "~" H 6100 6875 50  0001 C CNN
 	1    6100 6875
@@
 F 0 "R5" V 2225 6525 50  0000 C CNN
 F 1 "10K" V 2325 6525 50  0000 C CNN
-F 2 "" V 2255 6525 50  0001 C CNN
+F 2 "Resistor_SMD:R_0603_1608Metric" V 2255 6525 50  0001 C CNN
 F 3 "~" H 2325 6525 50  0001 C CNN
 	1    2325 6525
@@
 F 0 "J2" H 9920 2729 50  0000 R CNN
 F 1 "RJ45" H 9920 2820 50  0000 R CNN
-F 2 "" V 10250 2750 50  0001 C CNN
+F 2 "Connector_RJ:RJ45_Amphenol_54602-x08_Horizontal" V 10250 2750 50  0001 C CNN
 F 3 "~" V 10250 2750 50  0001 C CNN
 	1    10250 2725
@@
 U 1 1 5EB42735
 P 9500 3125
-F 0 "R21" V 9550 2975 50  0000 C CNN
+F 0 "R21" V 9550 2950 50  0000 C CNN
 F 1 "0" V 9500 3125 50  0000 C CNN
-F 2 "" V 9430 3125 50  0001 C CNN
+F 2 "Resistor_SMD:R_0603_1608Metric" V 9430 3125 50  0001 C CNN
 F 3 "~" H 9500 3125 50  0001 C CNN
 	1    9500 3125
@@
 U 1 1 5EB4D6BA
 P 9500 3025
-F 0 "R20" V 9550 2875 50  0000 C CNN
+F 0 "R20" V 9550 2850 50  0000 C CNN
 F 1 "0" V 9500 3025 50  0000 C CNN
-F 2 "" V 9430 3025 50  0001 C CNN
+F 2 "Resistor_SMD:R_0603_1608Metric" V 9430 3025 50  0001 C CNN
 F 3 "~" H 9500 3025 50  0001 C CNN
 	1    9500 3025
@@
 U 1 1 5EB4D95E
 P 9500 2925
-F 0 "R19" V 9550 2775 50  0000 C CNN
+F 0 "R19" V 9550 2750 50  0000 C CNN
 F 1 "0" V 9500 2925 50  0000 C CNN
-F 2 "" V 9430 2925 50  0001 C CNN
+F 2 "Resistor_SMD:R_0603_1608Metric" V 9430 2925 50  0001 C CNN
 F 3 "~" H 9500 2925 50  0001 C CNN
 	1    9500 2925
@@
 U 1 1 5EB4DC76
 P 9500 2825
-F 0 "R18" V 9550 2675 50  0000 C CNN
+F 0 "R18" V 9550 2650 50  0000 C CNN
 F 1 "0" V 9500 2825 50  0000 C CNN
-F 2 "" V 9430 2825 50  0001 C CNN
+F 2 "Resistor_SMD:R_0603_1608Metric" V 9430 2825 50  0001 C CNN
 F 3 "~" H 9500 2825 50  0001 C CNN
 	1    9500 2825
@@
 U 1 1 5EB4DED5
 P 9500 2725
-F 0 "R17" V 9550 2575 50  0000 C CNN
+F 0 "R17" V 9550 2550 50  0000 C CNN
 F 1 "0" V 9500 2725 50  0000 C CNN
-F 2 "" V 9430 2725 50  0001 C CNN
+F 2 "Resistor_SMD:R_0603_1608Metric" V 9430 2725 50  0001 C CNN
 F 3 "~" H 9500 2725 50  0001 C CNN
 	1    9500 2725
@@
 U 1 1 5EB4E167
 P 9500 2625
-F 0 "R16" V 9550 2475 50  0000 C CNN
+F 0 "R16" V 9550 2450 50  0000 C CNN
 F 1 "0" V 9500 2625 50  0000 C CNN
-F 2 "" V 9430 2625 50  0001 C CNN
+F 2 "Resistor_SMD:R_0603_1608Metric" V 9430 2625 50  0001 C CNN
 F 3 "~" H 9500 2625 50  0001 C CNN
 	1    9500 2625

Commit message: working on the PCB for the control board
Changed lines of the file:
@@
 Text Notes 1900 3650 0    50   ~ 0
 Relay Control Block 1
+Text HLabel 3000 4300 2    50   Input ~ 0
+Relay_Ouput1
 Text HLabel 3000 4200 2    50   Input ~ 0
-Relay_Ouput1
-Text HLabel 3000 4300 2    50   Input ~ 0
 Relay_Ouput2
 Text HLabel 5950 4625 2    50   Input ~ 0

Commit message: first pass of completed control board done
Connections:
- net labels removed: REED_SW1, REED_SW1_GND, REED_SW2, REED_SW2_GND
- wire segments 193 -> 191
Changed lines of the file:
@@
 	4025 1625 4125 1625
 NoConn ~ 6700 2550
-Text HLabel 6950 1750 2    50   Input ~ 0
-REED_SW1
 Wire Wire Line
 	6950 1750 6700 1750
-Text HLabel 6950 1850 2    50   Input ~ 0
-REED_SW2
 Wire Wire Line
 	6950 1850 6700 1850
@@
 Network Connected Microcontroller
 $Comp
-L FeatherWing_KC5-cache:+3.3V #PWR08
+L GarageDoorOpener-rescue:+3.3V-FeatherWing_KC5-cache #PWR08
 U 1 1 5EA9BBC7
 P 3775 1125
@@
 Text Notes 5950 5100 0    50   ~ 0
 REED SW2
-Text HLabel 4950 4625 0    50   Input ~ 0
-REED_SW1
-Text HLabel 4950 5250 0    50   Input ~ 0
-REED_SW2
 Wire Wire Line
 	4950 4625 5150 4625
-$Comp
-L power:GND #PWR?
-U 1 1 5EAF8DC4
-P 5850 5475
-AR Path="/5EAD635B/5EAF8DC4" Ref="#PWR?"  Part="1"
-AR Path="/5EAF8DC4" Ref="#PWR011"  Part="1"
-F 0 "#PWR011" H 5850 5225 50  0001 C CNN
-F 1 "GND" H 5855 5302 50  0000 C CNN
-F 2 "" H 5850 5475 50  0001 C CNN
-F 3 "" H 5850 5475 50  0001 C CNN
-	1    5850 5475
-	1    0    0    -1
-$EndComp
-Wire Wire Line
-	5850 5475 5850 5350
-Wire Wire Line
-	5850 5350 5950 5350
-Wire Wire Line
-	5950 4725 5850 4725
-Wire Wire Line
-	5850 4725 5850 5350
-Connection ~ 5850 5350
 $Comp
 L Device:R R?
@@
 	5150 4125 5150 4225
 $Comp
-L FeatherWing_KC5-cache:+3.3V #PWR?
+L GarageDoorOpener-rescue:+3.3V-FeatherWing_KC5-cache #PWR?
 U 1 1 5EAF8DDB
 P 5150 4075
@@
 $EndComp
 $Comp
-L FeatherWing_KC5-cache:+3.3V #PWR02
+L GarageDoorOpener-rescue:+3.3V-FeatherWing_KC5-cache #PWR02
 U 1 1 5EB006F0
 P 1325 3875
@@
 Text HLabel 5950 5250 2    50   Input ~ 0
 REED_SW2_IN
-Text HLabel 5950 4725 2    50   Input ~ 0
-REED_SW1_GND
-Text HLabel 5950 5350 2    50   Input ~ 0
-REED_SW2_GND
 Text HLabel 3850 2325 0    50   Input ~ 0
 LED_STRIP_CLK
@@
 	8950 4950 8450 4950
 $Comp
-L FeatherWing_KC5-cache:+3.3V #PWR017
+L GarageDoorOpener-rescue:+3.3V-FeatherWing_KC5-cache #PWR017
 U 1 1 5EB63A05
 P 8300 4100
@@
 $EndComp
 $Comp
-L FeatherWing_KC5-cache:+3.3V #PWR015
+L GarageDoorOpener-rescue:+3.3V-FeatherWing_KC5-cache #PWR015
 U 1 1 5EBB2CD0
 P 7525 3975
@@
 Text HLabel 9175 2825 0    50   Input ~ 0
 REED_SW2_IN
-Text HLabel 9175 2925 0    50   Input ~ 0
-REED_SW2_GND
-Text HLabel 9175 3025 0    50   Input ~ 0
+Text HLabel 8975 3025 0    50   Input ~ 0
 REED_SW1_IN
-Text HLabel 9175 3125 0    50   Input ~ 0
-REED_SW1_GND
 Text HLabel 9175 2625 0    50   Input ~ 0
 Relay_Ouput1
@@
 	9350 2825 9175 2825
 Wire Wire Line
-	9350 2925 9175 2925
-Wire Wire Line
-	9350 3025 9175 3025
+	9350 3025 8975 3025
 $Comp
 L Device:R R21
@@
 	0    1    1    0
 $EndComp
-Wire Wire Line
-	9350 3125 9175 3125
 $Comp
 L Device:R R20
@@
 	0    1    1    0
 $EndComp
+Text HLabel 4950 4625 0    50   Input ~ 0
+REED_SW1_IN
+Text HLabel 6950 1750 2    50   Input ~ 0
+REED_SW1_IN
+Text HLabel 4950 5250 0    50   Input ~ 0
+REED_SW2_IN
+Text HLabel 6950 1850 2    50   Input ~ 0
+REED_SW2_IN
+$Comp
+L power:GND #PWR?
+U 1 1 5EBC021D
+P 9100 3225
+F 0 "#PWR?" H 9100 2975 50  0001 C CNN
+F 1 "GND" H 9100 3075 50  0000 C CNN
+F 2 "" H 9100 3225 50  0001 C CNN
+F 3 "" H 9100 3225 50  0001 C CNN
+	1    9100 3225
+	1    0    0    -1
+$EndComp
+Wire Wire Line
+	9100 3225 9100 3125
+Wire Wire Line
+	9100 2925 9350 2925
+Wire Wire Line
+	9100 3125 9350 3125
+Connection ~ 9100 3125
+Wire Wire Line
+	9100 3125 9100 2925
 $EndSCHEMATC
